File: board/GWHP.kicad_pcb (KiCad board)
At the start: 2 copper layers, 57 parts, among them J1 Power Switch, J2 Mains, J3 AUX, J4 E2V, J5 LPS, J6 Pump Cold Side, J7 Pump Hot Side, J8 HPS, J9 Compressor, K1 RELAY_2, K2 RELAY_2, K3 RELAY_2, T1 MMBT3904, U1 NCP1117-3.3_SOT223, U10 LSA-TH3P, U2 NCP1117-3.3_SOT223, U3 Mean Well PM-15-5, U4 Omega2, U5 STM32F030K6Tx, U6 DRV8833, U7 DAC081C081, U8 G3MB-5V-SSR, U9 G3MB-5V-SSR, X1 SWD, X2 I2C Cold Side, X3 I2C Hot Side, X4 I2C Aux

Commit message: WIP
Parts:
- moved J2 324.3 mm to (179.5, 42.5), turned to 180 degrees
- moved K3 295.6 mm to (185.2, 109.9), turned to 180 degrees
- moved K1 268.8 mm to (185.2, 59.9), turned to 180 degrees
- moved U3 253.7 mm to (217.5, 70.0), turned to 180 degrees
- moved K2 253.3 mm to (185.3, 84.9), turned to 180 degrees
- moved U10 176.2 mm to (100.0, 92.5), turned to 270 degrees
- moved J5 172.6 mm to (120.0, 163.2)
- moved U2 167.3 mm to (370.6, 92.7)
- moved C10 156.1 mm to (364.8, 126.9)
- moved C2 156.1 mm to (347.6, 140.2)
- moved C8 156.1 mm to (339.8, 152.1)
- moved C9 156.1 mm to (351.7, 140.2)
- moved R11 156.1 mm to (360.9, 125.8)
- moved R8 156.1 mm to (365.3, 121.6)
- moved T1 156.1 mm to (341.5, 140.6)
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Connections:
- J2 pad 1: /MAINS_N -> /MAINS_L3
- J2 pad 2: /MAINS_L1 -> /MAINS_L2
- J2 pad 3: /MAINS_L2 -> /MAINS_L1
- J2 pad 4: /MAINS_L3 -> /MAINS_N
Routing:
- net (no net): vias 0 -> 6
Other:
- board outline added: 200 x 160 mm

Commit message: WIP
Parts:
- added D2: SK22, Diodes_SMD:D_SMB, F.Cu at (183.2, 134.0)
- added R16: 4R7/2W, Resistors_SMD:R_2512, F.Cu at (180.0, 125.6)
- added R17: 4R7/2W, Resistors_SMD:R_2512, F.Cu at (190.0, 125.6)
- added R18: 4R7/2W, Resistors_SMD:R_2512, F.Cu at (185.0, 125.6)
- moved R13 221.0 mm to (129.1, 156.0), turned to 180 degrees
- moved R12 207.8 mm to (129.1, 159.0)
- moved R15 200.2 mm to (143.9, 156.0), turned to 180 degrees
- moved R14 199.8 mm to (144.1, 159.0)
- moved U2 178.0 mm to (194.0, 114.8), turned to 270 degrees
- moved U1 171.6 mm to (194.0, 136.8), turned to 270 degrees
- moved D1 150.6 mm to (195.0, 125.8), turned to 90 degrees
- moved C2 148.6 mm to (199.0, 137.0), turned to 270 degrees
- moved C3 134.6 mm to (199.0, 115.0), turned to 270 degrees
- moved R7 82.6 mm to (311.0, 159.0)
- moved R4 78.8 mm to (302.1, 143.0)
- moved X1 53.5 mm to (289.0, 105.0)
- moved R5 50.6 mm to (308.1, 143.0)
- moved R3 50.0 mm to (304.0, 138.0)
- moved C8 47.2 mm to (381.0, 129.0)
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- renumbered D2 to D4
Connections:
- C1 pad 1: /5V_BACKUP -> Net-(C1-Pad1)
- D1 pad 2: +5V -> Net-(D1-Pad2)
- R1 pad 1: +5V -> (no net)

Commit message: WIP
Parts:
- moved S1 218.0 mm to (242.0, 220.0)
- moved R1 217.1 mm to (242.1, 225.0), turned to 180 degrees
- moved R2 210.7 mm to (242.1, 223.0)
- moved R8 198.2 mm to (199.0, 211.1), turned to 90 degrees
- moved R9 196.9 mm to (199.0, 215.1), turned to 270 degrees
- moved C11 190.0 mm to (173.0, 197.0), turned to 270 degrees
- moved C5 188.1 mm to (214.0, 213.0), turned to 270 degrees
- moved C7 185.3 mm to (235.0, 205.0)
- moved C8 185.2 mm to (214.0, 209.0), turned to 90 degrees
- moved C10 169.1 mm to (221.0, 216.0), turned to 90 degrees
- moved R11 165.3 mm to (198.9, 159.0)
- moved C4 157.3 mm to (235.0, 202.0)
- moved C6 140.0 mm to (214.0, 217.0), turned to 270 degrees
- moved C9 139.1 mm to (228.0, 204.0), turned to 180 degrees
- moved X1 136.1 mm to (237.5, 231.0)
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Connections:
- D1 pad 2: Net-(D1-Pad2) -> +5V
- R1 pad 1: (no net) -> +5V
- R16 pad 2: Net-(D1-Pad2) -> +5V
- R17 pad 2: Net-(D1-Pad2) -> +5V
- R18 pad 2: Net-(D1-Pad2) -> +5V
Other:
- outline, holes or cut-outs redrawn

Commit message: WIP
Parts:
- moved X1 2.89 mm to (239.5, 233.0)
- moved R1 1.00 mm to (242.1, 226.0)
- moved R2 1.00 mm to (242.1, 224.0)
- moved S1 1.00 mm to (242.0, 219.0)
Changed lines of the file:
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@@
     (links 191)
     (no_connects 191)
-    (area 44.924999 22.424999 245.075001 182.575001)
+    (area 72.924999 80.424999 273.075001 240.575001)
     (thickness 1.6)
     (drawings 20)
@@
   )
   (module Resistors_SMD:R_0805 (layer F.Cu)
-    (at 242.05 225 180)
+    (at 242.05 226 180)
     (descr "Resistor SMD 0805, reflow soldering, Vishay (see dcrcw.pdf)")
     (tags "resistor 0805")
@@
   )
   (module Resistors_SMD:R_0805 (layer F.Cu)
-    (at 242.05 223)
+    (at 242.05 224)
     (descr "Resistor SMD 0805, reflow soldering, Vishay (see dcrcw.pdf)")
     (tags "resistor 0805")
@@
   )
   (module device.farm:SB2P (layer F.Cu)
-    (at 242.016 220)
+    (at 242.016 219)
     (fp_text reference S1 (at 0 2.032) (layer F.SilkS)
       (effects (font (size 1 1) (thickness 0.15)))
@@
   )
   (module device.farm:SWD (layer F.Cu)
-    (at 237.46 231)
+    (at 239.54 233)
     (fp_text reference X1 (at 0 2.54) (layer F.SilkS)
       (effects (font (size 1 1) (thickness 0.15)))
@@
   )
   (dimension 200 (width 0.3) (layer Dwgs.User)
-    (gr_text "200,000 mm" (at 173 58.15) (layer Dwgs.User)
+    (gr_text "200,000 mm" (at 173 62.65) (layer Dwgs.User)
       (effects (font (size 1.5 1.5) (thickness 0.3)))
     )
-    (feature1 (pts (xy 273 80.5) (xy 273 56.8)))
-    (feature2 (pts (xy 73 80.5) (xy 73 56.8)))
-    (crossbar (pts (xy 73 59.5) (xy 273 59.5)))
-    (arrow1a (pts (xy 273 59.5) (xy 271.873496 60.086421)))
-    (arrow1b (pts (xy 273 59.5) (xy 271.873496 58.913579)))
-    (arrow2a (pts (xy 73 59.5) (xy 74.126504 60.086421)))
-    (arrow2b (pts (xy 73 59.5) (xy 74.126504 58.913579)))
+    (feature1 (pts (xy 273 80.5) (xy 273 61.3)))
+    (feature2 (pts (xy 73 80.5) (xy 73 61.3)))
+    (crossbar (pts (xy 73 64) (xy 273 64)))
+    (arrow1a (pts (xy 273 64) (xy 271.873496 64.586421)))
+    (arrow1b (pts (xy 273 64) (xy 271.873496 63.413579)))
+    (arrow2a (pts (xy 73 64) (xy 74.126504 64.586421)))
+    (arrow2b (pts (xy 73 64) (xy 74.126504 63.413579)))
   )
   (gr_line (start 73 85.5) (end 73 235.5) (layer Edge.Cuts) (width 0.15))

Commit message: WIP
Parts:
- moved R12 3.00 mm to (174.1, 217.0)
- moved R13 3.00 mm to (174.1, 214.0)
- moved R14 3.00 mm to (189.1, 217.0)
- moved R15 3.00 mm to (188.9, 214.0)
Changed lines of the file:
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@@
     (46 B.CrtYd user)
     (47 F.CrtYd user)
-    (48 B.Fab user)
-    (49 F.Fab user)
+    (48 B.Fab user hide)
+    (49 F.Fab user hide)
   )
   (setup
@@
     (pad_to_mask_clearance 0.2)
     (aux_axis_origin 0 0)
-    (visible_elements FFFFEF7F)
+    (visible_elements FFFEEF7F)
     (pcbplotparams
       (layerselection 0x00030_80000001)
@@
   )
   (module Resistors_SMD:R_0805 (layer F.Cu)
-    (at 171.05 217)
+    (at 174.05 217)
     (descr "Resistor SMD 0805, reflow soldering, Vishay (see dcrcw.pdf)")
     (tags "resistor 0805")
@@
   )
   (module Resistors_SMD:R_0805 (layer F.Cu)
-    (at 171.05 214 180)
+    (at 174.05 214 180)
     (descr "Resistor SMD 0805, reflow soldering, Vishay (see dcrcw.pdf)")
     (tags "resistor 0805")
@@
   )
   (module Resistors_SMD:R_0805 (layer F.Cu)
-    (at 186.05 217)
+    (at 189.05 217)
     (descr "Resistor SMD 0805, reflow soldering, Vishay (see dcrcw.pdf)")
     (tags "resistor 0805")
@@
   )
   (module Resistors_SMD:R_0805 (layer F.Cu)
-    (at 185.95 214 180)
+    (at 188.95 214 180)
     (descr "Resistor SMD 0805, reflow soldering, Vishay (see dcrcw.pdf)")
     (tags "resistor 0805")

Commit message: WIP
Parts:
- moved J3 10.5 mm to (244.0, 213.0), turned to 180 degrees
Connections:
- J3 pad 2: GND -> Net-(J3-Pad2)
- J3 pad 4: GND -> Net-(J3-Pad4)
- J3 pad 5: +3V3 -> GND
- J3 pad 7: Net-(J3-Pad7) -> GND
- J3 pad 9: Net-(J3-Pad9) -> +3V3
- U5 pad 27: Net-(J3-Pad9) -> Net-(J3-Pad2)
- U5 pad 28: Net-(J3-Pad8) -> Net-(J3-Pad4)
- U5 pad 29: Net-(J3-Pad7) -> Net-(J3-Pad6)
- U5 pad 30: Net-(J3-Pad6) -> Net-(J3-Pad8)
Routing:
- net /COMP_L1: track 0.00 -> 216.1 mm
- net /COMP_L3: track 0.00 -> 199.7 mm
- net /COMP_L2: track 0.00 -> 194.5 mm
- net /MAINS_L3: track 0.00 -> 134.6 mm
- net /MAINS_L2: track 0.00 -> 116.1 mm
- net /MAINS_L1: track 0.00 -> 68.1 mm
- net (no net): vias 6 -> 0
Other:
- net class Default: trace_width 0.25 -> 0.4
- net class HC added: clearance 1.5, trace_width 4.5, via_dia 4.5, via_drill 2
- net class PWR added: clearance 0.2, trace_width 0.6, via_dia 0.9, via_drill 0.6

Commit message: WIP
Parts:
- moved J1 124.7 mm to (84.5, 221.6), turned to 0 degrees
- moved R16 25.3 mm to (188.0, 199.1)
- moved R17 25.3 mm to (198.0, 199.1)
- moved R18 25.3 mm to (193.0, 199.1)
- moved R11 25.3 mm to (221.6, 170.3), turned to 90 degrees
- moved D1 20.5 mm to (209.0, 198.8)
- moved D3 15.0 mm to (212.6, 171.5), turned to 90 degrees
- moved K3 14.9 mm to (212.4, 153.0)
- moved C1 14.2 mm to (200.0, 182.0)
- moved C11 13.5 mm to (180.0, 208.5)
- moved U7 13.5 mm to (184.6, 208.6)
- moved T1 12.7 mm to (217.6, 170.3), turned to 180 degrees
- moved D2 10.6 mm to (203.0, 198.8), turned to 90 degrees
- moved U2 9.11 mm to (219.3, 181.6)
- moved C3 9.11 mm to (224.3, 181.7)
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Connections:
- J1 pad 2: Net-(J1-Pad2) -> /SWITCHED_L
- J9 pad 1: /COMP_L1 -> /COMP_L3
- J9 pad 3: /COMP_L3 -> /COMP_L1
- U10 pad 7: /MAINS_L1 -> /SWITCHED_L
- U3 pad 1: Net-(J1-Pad2) -> /SWITCHED_L
- U8 pad 1: /MAINS_L1 -> /SWITCHED_L
- U9 pad 1: /MAINS_L1 -> /SWITCHED_L
Routing:
- net /MAINS_N: track 0.00 -> 297.2 mm, vias 0 -> 3
- net /SWITCHED_L: track 0.00 -> 284.3 mm
- net /MAINS_L1: track 68.1 -> 198.5 mm, vias 0 -> 1
- net Net-(J7-Pad2): track 0.00 -> 25.1 mm
- net /MAINS_L2: track 116.1 -> 93.9 mm
- net Net-(J6-Pad2): track 0.00 -> 21.7 mm
- net /COMP_L1: track 216.1 -> 236.1 mm
- net /COMP_L3: track 199.7 -> 180.3 mm
- net /COMP_L2: track 194.5 -> 209.4 mm
- net /MAINS_L3: track 134.6 -> 130.6 mm
- net (no net): vias 0 -> 6
- added copper zone on B.Cu, net GND

Commit message: WIP
Parts:
- added J10: Service, Pin_Headers:Pin_Header_Straight_1x06_Pitch2.54mm, F.Cu at (268.0, 215.7)
- added REF**: MountingHole_3.7mm_Pad, Mounting_Holes:MountingHole_3.7mm_Pad, F.Cu at (268.0, 236.0)
- added REF**: MountingHole_3.7mm_Pad, Mounting_Holes:MountingHole_3.7mm_Pad, F.Cu at (177.0, 199.0)
- added REF**: MountingHole_3.7mm_Pad, Mounting_Holes:MountingHole_3.7mm_Pad, F.Cu at (78.0, 236.0)
- added REF**: MountingHole_3.7mm_Pad, Mounting_Holes:MountingHole_3.7mm_Pad, F.Cu at (268.0, 86.0)
- added REF**: MountingHole_3.7mm_Pad, Mounting_Holes:MountingHole_3.7mm_Pad, F.Cu at (158.7, 88.7)
- added REF**: MountingHole_3.7mm_Pad, Mounting_Holes:MountingHole_3.7mm_Pad, F.Cu at (78.0, 86.0)
- moved C11 85.9 mm to (265.0, 221.0), turned to 180 degrees
- moved U7 84.1 mm to (267.0, 225.6), turned to 270 degrees
- moved X4 1.25 mm to (256.0, 207.0)
- moved X3 0.75 mm to (256.0, 219.0)
- moved J3 0.57 mm to (243.5, 213.2)
- moved X2 0.50 mm to (256.0, 231.0)
Connections:
- U4 pad 27: (no net) -> /TX0
- U4 pad 28: (no net) -> /RX0
- U4 pad 29: (no net) -> /USB-DM
- U4 pad 30: (no net) -> /USB-DP
Routing:
- net GND: track 0.00 -> 205.6 mm
- net Net-(U10-Pad11): track 0.00 -> 157.6 mm
- net /SWITCHED_L: track 284.3 -> 285.8 mm
- net /MAINS_N: track 297.2 -> 298.7 mm
- net (no net): vias 6 -> 0
