File: board/GWHP.kicad_pcb (KiCad board)
At the start: 2 copper layers, 200 x 160 mm, 68 parts, among them J1 Power Switch, J10 Service, J2 Mains, J3 AUX, J4 E2V, J5 LPS, J6 Pump Cold Side, J7 Pump Hot Side, J8 HPS, J9 Compressor, K1 RELAY_2, K2 RELAY_2, K3 RELAY_2, T1 MMBT3904, U1 NCP1117-3.3_SOT223, U10 LSA-TH3P, U2 NCP1117-3.3_SOT223, U3 Mean Well PM-15-5, U4 Omega2, U5 STM32F030K6Tx, U6 DRV8833, U7 DAC081C081, U8 G3MB-5V-SSR, U9 G3MB-5V-SSR, X1 SWD, X2 I2C Cold Side, X3 I2C Hot Side, X4 I2C Aux

Commit message: WIP
Parts:
- moved C11 1.00 mm to (266.0, 221.0)
- turned D1 to 270 degrees
- turned R16 to 270 degrees
- turned R17 to 270 degrees
- turned R18 to 270 degrees
Connections:
- net Net-(C1-Pad1) renamed /BACKUP_C
Routing:
- net GND: track 205.6 -> 312.7 mm, vias 0 -> 16
- net +5V: track 0.00 -> 92.6 mm
- net /SCL: track 0.00 -> 72.6 mm, vias 0 -> 4
- net /SDA: track 0.00 -> 70.2 mm, vias 0 -> 4
- net /5V_BACKUP: track 0.00 -> 53.3 mm
- net +3V3: track 0.00 -> 36.1 mm
- net /BACKUP_C: track 0.00 -> 32.3 mm
- net Net-(J5-Pad2): track 0.00 -> 31.2 mm
- net /E2V_A1: track 0.00 -> 30.2 mm, vias 0 -> 2
- net /ALERT: track 0.00 -> 30.1 mm
- net /E2V_A2: track 0.00 -> 29.9 mm, vias 0 -> 2
- net /E2V_B2: track 0.00 -> 28.7 mm, vias 0 -> 2
- net /E2V_NFAULT: track 0.00 -> 28.4 mm, vias 0 -> 2
- net /E2V_NSLEEP: track 0.00 -> 26.8 mm, vias 0 -> 2
- net /E2V_B1: track 0.00 -> 25.6 mm, vias 0 -> 2
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Other:
- net class Default: clearance 0.2 -> 0.199
- net class PWR: clearance 0.2 -> 0.199
- rule trace_clearance: 0.2 -> 0.199

Commit message: WIP
Parts:
- moved R11 2.97 mm to (224.5, 170.0), turned to 270 degrees
- moved T1 2.97 mm to (220.5, 170.0)
- moved D3 2.01 mm to (213.8, 170.0), turned to 0 degrees
Connections:
- net Net-(D3-Pad2) renamed /COMP_RELAY_PWR
Routing:
- net /COMP_5V: track 19.7 -> 252.2 mm, vias 0 -> 3
- net +5V: track 92.6 -> 236.3 mm, vias 0 -> 5
- net Net-(U10-Pad11): track 157.6 -> 285.1 mm
- net /PUMP_HOT_SIDE: track 0.00 -> 119.5 mm, vias 0 -> 2
- net /PUMP_COLD_SIDE: track 0.00 -> 107.0 mm
- net /COMP_RELAY_PWR: track 0.00 -> 63.5 mm, vias 0 -> 1
- net /SCL: track 72.6 -> 97.3 mm, vias 4 -> 6
- net /SDA: track 70.2 -> 93.7 mm, vias 4 -> 6
- net /PWR_OK: track 0.00 -> 18.0 mm, vias 0 -> 2
- net /3V3_BACKUP: track 25.3 -> 41.3 mm
- net +3V3: track 36.1 -> 40.1 mm
- net Net-(R11-Pad1): track 0.00 -> 3.79 mm
- net /SWDIO: track 19.1 -> 19.9 mm

Commit message: WIP
Routing:
- net +3V3: track 40.1 -> 157.5 mm, vias 0 -> 2
- net /LPS: track 3.00 -> 73.1 mm, vias 0 -> 2
- net /HPS: track 3.04 -> 60.1 mm, vias 0 -> 2
- net /ALERT: track 30.1 -> 87.1 mm, vias 0 -> 5
- net /COMP_RELAY: track 0.00 -> 53.1 mm, vias 0 -> 2
- net /3V3_BACKUP: track 41.3 -> 91.2 mm, vias 0 -> 5
- net /5V_BACKUP: track 53.3 -> 68.9 mm
- net Net-(R5-Pad1): track 0.00 -> 11.1 mm, vias 0 -> 2
- net Net-(C4-Pad1): track 0.00 -> 7.55 mm
- net +5V: track 236.3 -> 232.2 mm, vias 5 -> 7
- net GND: track 312.6 -> 314.9 mm, vias 16 -> 17
- net /USB-DP: track 13.5 -> 15.3 mm
- net /PUMP_HOT_SIDE: track 119.5 -> 120.6 mm
- net /USB-DM: track 16.8 -> 17.7 mm
- net /TX0: track 23.6 -> 24.3 mm
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
Commit message: WIP
Routing:
- net /SWITCHED_L: track 285.8 -> 293.4 mm
- net /MAINS_L1: track 198.5 -> 206.1 mm
- net GND: track 314.9 -> 315.8 mm
- net /E2V_B2: track 28.7 -> 28.1 mm
- net /E2V_A2: track 29.8 -> 29.3 mm
Other:
- board text added: "5V"
- board text added: "A1"
- board text added: "A2"
- board text added: "AUX"
- board text added: "B1"
- board text added: "B2"
- board text added: "CC-BY-NC-SA"
- board text added: "COMPRESSOR"
- board text added: "D+"
- board text added: "D-"
- board text added: "DEVICE.FARM"
- board text added: "EXPANSION VALVE"
- board text added: "GND"
- board text added: "GWHP v1.0"
- board text added: "HIGH PRESSURE"
- board text added: "I2C"
- board text added: "L1"
- board text added: "L2"
- board text added: "L3"
- board text added: "LOW PRESSURE"
- board text added: "MAIN SWITCH"
- board text added: "MAINS"
- board text added: "N"
- board text added: "PUMP COLD SIDE"
- board text added: "PUMP HOT SIDE"
- board text added: "RX0"
- board text added: "SERVICE"
- board text added: "SWD"
- board text added: "TX0"
- board text added: "WARNING HIGH VOLTAGE"

Commit message: WIP
Parts:
- added C12: 100n, Capacitors_SMD:C_0805, F.Cu at (173.0, 251.1)
- C5: value 100n -> 10M
- U6: footprint Housings_SSOP:TSSOP-16_4.4x5mm_Pitch0.65mm -> device.farm:TSSOP-16_4.4x5mm_Pitch0.65mm-EP
- U7: value DAC081C081 -> MCP4706A0T-E/CH
- moved J1 32.4 mm to (116.9, 221.6)
- moved J9 14.5 mm to (90.5, 223.0)
- moved REF** 9.67 mm to (168.0, 86.0)
- moved U10 5.00 mm to (128.0, 144.0)
- moved K3 1.08 mm to (212.0, 154.0)
- moved K1 0.55 mm to (212.0, 114.0)
- moved K2 0.40 mm to (212.0, 134.0)
- turned C11 to 0 degrees
Connections:
- U7 pad 2: /COMP_5V -> GND
- U7 pad 3: GND -> /COMP_5V
- U7 pad 6: GND -> (no net)
Routing:
- net /SWITCHED_L: track 293.4 -> 8.00 mm
- net /COMP_L1: track 236.1 -> 0.00 mm
- net /COMP_L2: track 209.4 -> 0.00 mm
- net /MAINS_L1: track 206.1 -> 0.00 mm, vias 1 -> 0
- net /MAINS_N: track 298.1 -> 115.4 mm, vias 2 -> 0
- net /COMP_L3: track 180.3 -> 0.00 mm
- net /MAINS_L3: track 130.6 -> 0.00 mm
- net /MAINS_L2: track 93.9 -> 0.00 mm
- net GND: track 315.8 -> 372.0 mm, vias 17 -> 20
- net /E2V_A2: track 29.3 -> 3.50 mm, vias 2 -> 0
- net /E2V_B2: track 28.1 -> 4.69 mm, vias 2 -> 0
- net /COMP_5V: track 252.4 -> 238.7 mm
- net /COMP_RELAY_PWR: track 63.5 -> 50.7 mm
- net /5V_BACKUP: track 68.9 -> 59.7 mm
Other:
- net class HC: trace_width 4.5 -> 4; via_dia 4.5 -> 4
- board text added: "GWHP v1.1"
- board text removed: "GWHP v1.0"

Commit message: WIP
Parts:
- removed the REF** at (177.0, 199.0)
- removed the REF** at (168.0, 86.0)
- removed U10: LSA-TH3P, device.farm:LSA-TH3P
- added J11: Mains L3, device.farm:Tab-6.3, F.Cu at (155.0, 132.5)
- added J12: Mains N, device.farm:Tab-6.3, F.Cu at (165.0, 132.5)
- added J13: SSR 220, device.farm:DG142R-2-5.08, F.Cu at (202.5, 139.8)
- added J14: SSR 0-5V, device.farm:DG142R-2-5.08, F.Cu at (242.5, 139.8)
- added J15: Compressor L1, device.farm:Tab-6.3, F.Cu at (115.0, 227.5)
- added J16: Compressor L2, device.farm:Tab-6.3, F.Cu at (135.0, 227.5)
- added J17: Compressor L3, device.farm:Tab-6.3, F.Cu at (155.0, 227.5)
- added J18: SSR Output L1, device.farm:Tab-6.3, F.Cu at (105.0, 227.5)
- added J19: SSR Output L2, device.farm:Tab-6.3, F.Cu at (125.0, 227.5)
- added J20: SSR Output L3, device.farm:Tab-6.3, F.Cu at (145.0, 227.5)
- added J21: SSR Input L1, device.farm:Tab-6.3, F.Cu at (105.0, 132.5)
- added J22: SSR Input L2, device.farm:Tab-6.3, F.Cu at (125.0, 132.5)
- added J23: SSR Input L3, device.farm:Tab-6.3, F.Cu at (145.0, 132.5)
- J2: value Mains -> Mains L1; footprint device.farm:HB-9500-4P -> device.farm:Tab-6.3
- J9: value Compressor -> Mains L2; footprint device.farm:HB-9500-3P -> device.farm:Tab-6.3
- T1: value MMBT3904 -> BC817
- moved U3 135.3 mm to (125.0, 190.0), turned to 270 degrees
- moved J1 108.1 mm to (187.5, 139.8), turned to 180 degrees
- moved K1 102.6 mm to (115.0, 147.4)
- moved J9 100.9 mm to (135.0, 132.5), turned to 90 degrees
- moved J2 97.7 mm to (115.0, 132.5), turned to 90 degrees
- moved C11 89.8 mm to (248.0, 133.0)
- moved U7 89.7 mm to (247.9, 137.9)
- moved C12 80.2 mm to (240.0, 207.0), turned to 90 degrees
- moved K2 63.4 mm to (150.0, 147.4)
- moved X1 58.8 mm to (231.1, 175.3), turned to 180 degrees
- moved C3 53.1 mm to (172.8, 169.1), turned to 0 degrees
- moved C1 52.5 mm to (216.0, 132.0), turned to 180 degrees
- moved J10 49.9 mm to (238.8, 175.3), turned to 90 degrees
- moved D1 48.2 mm to (213.0, 150.8)
- moved D2 48.2 mm to (207.0, 150.8)
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Connections:
- J1 pad 1: /MAINS_L1 -> /SWITCHED_L
- J1 pad 2: /SWITCHED_L -> /MAINS_L1
- J2 pad 1: /MAINS_L3 -> /MAINS_L1
- J9 pad 1: /COMP_L3 -> /MAINS_L2
- U7 pad 1: Net-(U10-Pad11) -> /COMP_RAMP
- U8 pad 1: /SWITCHED_L -> Net-(J6-Pad2)
- U8 pad 2: Net-(J6-Pad2) -> /SWITCHED_L
- U9 pad 1: /SWITCHED_L -> Net-(J7-Pad2)
- U9 pad 2: Net-(J7-Pad2) -> /SWITCHED_L
Routing:
- net GND: track 372.0 -> 0.00 mm, vias 20 -> 0
- net Net-(U10-Pad11): track 285.1 -> 0.00 mm
- net /COMP_5V: track 238.7 -> 0.00 mm, vias 3 -> 0
- net +5V: track 232.2 -> 0.00 mm, vias 7 -> 0
- net +3V3: track 157.5 -> 0.00 mm, vias 2 -> 0
- net /PUMP_HOT_SIDE: track 120.6 -> 0.00 mm, vias 2 -> 0
- net /MAINS_N: track 115.4 -> 0.00 mm
- net /PUMP_COLD_SIDE: track 107.7 -> 0.00 mm
- net /SCL: track 97.4 -> 0.00 mm, vias 6 -> 0
- net /SDA: track 94.4 -> 0.00 mm, vias 6 -> 0
- net /3V3_BACKUP: track 91.2 -> 0.00 mm, vias 5 -> 0
- net /ALERT: track 87.1 -> 0.00 mm, vias 5 -> 0
- net /LPS: track 73.1 -> 0.00 mm, vias 2 -> 0
- net /HPS: track 60.1 -> 0.00 mm, vias 2 -> 0
- net /5V_BACKUP: track 59.7 -> 0.00 mm
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- removed copper zone on B.Cu, net GND
Other:
- board size 200 x 160 mm -> 175 x 120 mm

Commit message: WIP
Parts:
- added C13: 2F, device.farm:BCE005R5C205FS, F.Cu at (204.5, 153.0)
- moved D1 28.0 mm to (190.0, 166.8)
- moved D2 28.0 mm to (184.0, 166.8)
- moved R16 28.0 mm to (169.0, 167.1)
- moved R17 28.0 mm to (179.0, 167.1)
- moved R18 28.0 mm to (174.0, 167.1)
- moved R11 26.4 mm to (198.0, 180.9)
- moved T1 14.7 mm to (197.9, 176.0), turned to 90 degrees
- moved C2 8.25 mm to (186.8, 177.1)
- moved C3 8.25 mm to (174.8, 177.1)
- moved U1 8.25 mm to (186.6, 182.1)
- moved U2 8.25 mm to (174.6, 182.1)
- moved D3 5.01 mm to (200.2, 169.0), turned to 180 degrees
- moved J12 2.90 mm to (166.5, 130.0), turned to 180 degrees
- moved C9 1.42 mm to (206.0, 191.0), turned to 180 degrees
Connections:
- K1 pad 12: (no net) -> /MAINS_L1
- K1 pad 22: (no net) -> /MAINS_L1
- K2 pad 12: (no net) -> /MAINS_L2
- K2 pad 22: (no net) -> /MAINS_L2
- K3 pad 12: (no net) -> /MAINS_L3
- K3 pad 22: (no net) -> /MAINS_L3
Routing:
- net /MAINS_L1: track 0.00 -> 154.4 mm
- net /COMP_L3: track 0.00 -> 141.2 mm, vias 0 -> 1
- net /COMP_L1: track 0.00 -> 127.9 mm, vias 0 -> 1
- net /COMP_L2: track 0.00 -> 121.1 mm, vias 0 -> 1
- net /MAINS_L3: track 0.00 -> 78.0 mm
- net /MAINS_L2: track 0.00 -> 70.6 mm
- net /MAINS_N: track 0.00 -> 50.1 mm
- net /SWITCHED_L: track 0.00 -> 15.2 mm
Other:
- net class Default: clearance 0.199 -> 0.2
- net class HC: clearance 1.5 -> 1.4; trace_width 4 -> 5
- net class LC added: clearance 1, trace_width 1, via_dia 1, via_drill 0.6
- net class PWR: clearance 0.199 -> 0.2
- rule trace_clearance: 0.199 -> 0.2

Commit message: WIP
Parts:
- moved R10 45.3 mm to (256.0, 219.9), turned to 90 degrees
- moved R6 41.8 mm to (253.0, 219.9), turned to 90 degrees
- moved R7 38.3 mm to (250.0, 219.9), turned to 90 degrees
- moved R2 20.4 mm to (257.0, 179.9), turned to 270 degrees
- moved R1 17.9 mm to (257.0, 175.9), turned to 270 degrees
- moved S1 2.31 mm to (220.0, 177.0)
- moved R8 1.15 mm to (223.9, 206.0), turned to 0 degrees
- moved R9 1.15 mm to (223.9, 209.0), turned to 0 degrees
- moved R11 1.00 mm to (197.0, 180.9)
- moved R13 0.10 mm to (201.6, 211.9)
- turned C5 to 270 degrees
Routing:
- net /MAINS_N: track 50.1 -> 322.6 mm, vias 0 -> 1
- net /COMP_5V: track 0.00 -> 194.5 mm, vias 0 -> 2
- net /SWITCHED_L: track 15.2 -> 204.0 mm, vias 0 -> 1
- net +3V3: track 0.00 -> 168.1 mm, vias 0 -> 5
- net /COMP_RELAY_PWR: track 0.00 -> 152.4 mm, vias 0 -> 1
- net /SDA: track 0.00 -> 132.0 mm, vias 0 -> 2
- net /SCL: track 0.00 -> 128.5 mm, vias 0 -> 2
- net /LPS: track 0.00 -> 108.3 mm, vias 0 -> 2
- net GND: track 0.00 -> 104.9 mm, vias 0 -> 32
- net /ALERT: track 0.00 -> 93.7 mm, vias 0 -> 4
- net +5V: track 0.00 -> 93.6 mm
- net /HPS: track 0.00 -> 89.7 mm, vias 0 -> 2
- net /BACKUP_C: track 0.00 -> 66.1 mm
- net /5V_BACKUP: track 0.00 -> 54.7 mm, vias 0 -> 2
- net /3V3_BACKUP: track 0.00 -> 50.0 mm
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- added copper zone on B.Cu, net GND
Other:
- net class Default: clearance 0.2 -> 0.199
- net class LC: via_dia 1 -> 1.2; via_drill 0.6 -> 0.8
- net class PWR: clearance 0.2 -> 0.199
- rule trace_clearance: 0.2 -> 0.199
