File: board/GWHP.kicad_pcb (KiCad board)
At the start: 2 copper layers, 175 x 120 mm, 80 parts, among them J1 Power Switch, J10 Service, J11 Mains L3, J12 Mains N, J13 SSR 220, J14 SSR 0-5V, J15 Compressor L1, J16 Compressor L2, J17 Compressor L3, J18 SSR Output L1, J19 SSR Output L2, J2 Mains L1, J20 SSR Output L3, J21 SSR Input L1, J22 SSR Input L2, J23 SSR Input L3, J3 AUX, J4 E2V, J5 LPS, J6 Pump Cold Side, J7 Pump Hot Side, J8 HPS, J9 Mains L2, K1 RELAY_2, K2 RELAY_2, K3 RELAY_2, T1 BC817, U1 NCP1117-3.3_SOT223, U2 NCP1117-3.3_SOT223, U3 Mean Well PM-15-5, U4 Omega2, U5 STM32F030K6Tx, U6 DRV8833, U7 MCP4706A0T-E/CH, U8 G3MB-5V-SSR, U9 G3MB-5V-SSR, X1 SWD, X2 I2C Cold Side, X3 I2C Hot Side, X4 I2C Aux

Commit message: WIP
Routing:
- net +5V: track 93.6 -> 271.8 mm, vias 0 -> 7
- net /COMP_5V: track 194.5 -> 345.8 mm, vias 2 -> 4
- net /3V3_BACKUP: track 50.0 -> 142.8 mm, vias 0 -> 4
- net /5V_BACKUP: track 54.7 -> 135.8 mm, vias 2 -> 6
- net GND: track 104.9 -> 106.8 mm, vias 32 -> 33
- net /PUMP_COLD_SIDE: track 42.3 -> 40.8 mm
- net /E2V_NFAULT: track 30.7 -> 31.8 mm

Commit message: WIP
Routing:
- net +5V: track 271.8 -> 271.0 mm
- net /5V_BACKUP: track 135.8 -> 135.2 mm
Changed lines of the file:
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@@
   (general
     (links 224)
-    (no_connects 3)
+    (no_connects 0)
     (area 84.924999 119.924999 260.075001 240.075001)
     (thickness 1.6)
@@
   (module device.farm:DG142R-2-5.08 (layer F.Cu)
     (at 242.54 139.778 180)
-    (fp_text reference J14 (at 5.334 15.494 180) (layer F.SilkS)
+    (fp_text reference J14 (at -3.46 15.778 180) (layer F.SilkS)
       (effects (font (size 1 1) (thickness 0.15)))
     )
@@
     (effects (font (size 1.5 1.5) (thickness 0.3)))
   )
-  (gr_text I2C (at 272.5 156) (layer F.SilkS)
+  (gr_text I2C (at 245 211) (layer F.SilkS)
     (effects (font (size 1.5 1.5) (thickness 0.3)))
   )
-  (gr_text I2C (at 272.5 168) (layer F.SilkS)
+  (gr_text I2C (at 245 199) (layer F.SilkS)
     (effects (font (size 1.5 1.5) (thickness 0.3)))
   )
-  (gr_text I2C (at 272.5 180) (layer F.SilkS)
+  (gr_text I2C (at 245 187) (layer F.SilkS)
     (effects (font (size 1.5 1.5) (thickness 0.3)))
   )
@@
     (effects (font (size 1.5 1.5) (thickness 0.3)))
   )
-  (gr_text "MAIN\nSWITCH" (at 242 103) (layer F.SilkS)
+  (gr_text "MAIN\nSWITCH" (at 237 123 180) (layer F.SilkS)
     (effects (font (size 1.5 1.5) (thickness 0.3)))
   )
@@
   (gr_line (start 260 125) (end 260 235) (layer Edge.Cuts) (width 0.15))
   (gr_line (start 255 120) (end 90 120) (layer Edge.Cuts) (width 0.15))
+  (segment (start 190 164.7) (end 190.708101 164.7) (width 0.6) (layer F.Cu) (net 1))
+  (segment (start 190.708101 164.7) (end 194.036735 168.028634) (width 0.6) (layer F.Cu) (net 1))
+  (segment (start 194.036735 168.028634) (end 194.036735 171.079682) (width 0.6) (layer F.Cu) (net 1))
+  (segment (start 194.036735 171.079682) (end 194.036735 171.716078) (width 0.6) (layer F.Cu) (net 1))
+  (segment (start 194 174) (end 194 171.752813) (width 0.6) (layer B.Cu) (net 1))
+  (segment (start 194 171.752813) (end 194.036735 171.716078) (width 0.6) (layer B.Cu) (net 1))
+  (via (at 194.036735 171.716078) (size 0.9) (drill 0.6) (layers F.Cu B.Cu) (net 1))
   (segment (start 188.288925 191.239991) (end 188.738924 191.68999) (width 0.6) (layer B.Cu) (net 1))
   (segment (start 186 188.951066) (end 188.288925 191.239991) (width 0.6) (layer B.Cu) (net 1))
@@
   (segment (start 185.428234 184.428234) (end 186 185) (width 0.6) (layer F.Cu) (net 1))
   (via (at 186 185) (size 0.9) (drill 0.6) (layers F.Cu B.Cu) (net 1))
-  (segment (start 194 171) (end 194 166.95) (width 0.6) (layer F.Cu) (net 1))
-  (segment (start 194 166.95) (end 191.75 164.7) (width 0.6) (layer F.Cu) (net 1))
-  (segment (start 191.75 164.7) (end 190 164.7) (width 0.6) (layer F.Cu) (net 1))
-  (via (at 194 171) (size 0.9) (drill 0.6) (layers F.Cu B.Cu) (net 1))
-  (segment (start 194 174) (end 194 171) (width 0.6) (layer B.Cu) (net 1))
   (segment (start 181 174) (end 194 174) (width 0.6) (layer F.Cu) (net 1))
   (via (at 194 174) (size 0.9) (drill 0.6) (layers F.Cu B.Cu) (net 1))
@@
   (segment (start 115 147.38) (end 115 145.810504) (width 0.6) (layer F.Cu) (net 8))
   (segment (start 115 145.810504) (end 119.205494 141.60501) (width 0.6) (layer F.Cu) (net 8))
+  (segment (start 165.995604 199.004396) (end 158.469068 199.004396) (width 0.6) (layer F.Cu) (net 9))
+  (segment (start 158.469068 199.004396) (end 156 201.473464) (width 0.6) (layer F.Cu) (net 9))
+  (segment (start 156 201.473464) (end 156 201.5) (width 0.6) (layer F.Cu) (net 9))
+  (segment (start 253 176.8) (end 253.905 177.705) (width 0.6) (layer F.Cu) (net 9))
+  (segment (start 253.905 177.705) (end 253.905 182.65) (width 0.6) (layer F.Cu) (net 9))
+  (segment (start 253.905 182.65) (end 253.905 184.75) (width 0.6) (layer F.Cu) (net 9))
   (segment (start 165.995604 199.004396) (end 194.78238 199.004396) (width 0.6) (layer F.Cu) (net 9))
-  (segment (start 160.845604 199.004396) (end 165.995604 199.004396) (width 0.6) (layer F.Cu) (net 9))
   (segment (start 165.995604 199.004396) (end 166 199) (width 0.6) (layer F.Cu) (net 9))
   (segment (start 166 191.232332) (end 166 199) (width 0.6) (layer F.Cu) (net 9))
   (segment (start 196.5 222.38) (end 196.5 200.722016) (width 0.6) (layer F.Cu) (net 9))
   (segment (start 196.5 200.722016) (end 194.78238 199.004396) (width 0.6) (layer F.Cu) (net 9))
-  (segment (start 160.845604 199.004396) (end 158.35 201.5) (width 0.6) (layer F.Cu) (net 9))
-  (segment (start 158.35 201.5) (end 156 201.5) (width 0.6) (layer F.Cu) (net 9))
   (segment (start 174.503306 184.428234) (end 174.515434 184.440362) (width 0.6) (layer F.Cu) (net 9))
   (segment (start 171.454098 184.428234) (end 174.503306 184.428234) (width 0.6) (layer F.Cu) (net 9))
@@
   (segment (start 171.454098 184.428234) (end 171.454098 185.778234) (width 0.6) (layer F.Cu) (net 9))
   (segment (start 171.454098 184.428234) (end 171.204098 184.428234) (width 0.6) (layer F.Cu) (net 9))
-  (segment (start 253.905 182.65) (end 253.905 184.75) (width 0.6) (layer F.Cu) (net 9))
-  (segment (start 254.79901 178.59901) (end 254.79901 181.330962) (width 0.6) (layer F.Cu) (net 9))
-  (segment (start 253.905 182.224972) (end 253.905 182.65) (width 0.6) (layer F.Cu) (net 9))
-  (segment (start 254.79901 181.330962) (end 253.905 182.224972) (width 0.6) (layer F.Cu) (net 9))
-  (segment (start 253 176.8) (end 254.79901 178.59901) (width 0.6) (layer F.Cu) (net 9))
   (segment (start 251.46 175.26) (end 253 176.8) (width 0.6) (layer F.Cu) (net 9))
   (segment (start 257 175) (end 254.8 175) (width 0.6) (layer F.Cu) (net 9))

Commit message: WIP
Parts:
- added REF***: OSHW-Logo_11.4x12mm_SilkScreen, Symbols:OSHW-Logo_11.4x12mm_SilkScreen, F.Cu at (201.0, 198.0)
- moved J12 4.25 mm to (169.0, 133.5), turned to 270 degrees
Routing:
- net /MAINS_N: track 322.6 -> 329.1 mm
- net /MAINS_L1: track 154.4 -> 155.0 mm
Other:
- board text added: "!"
- board text added: "0-5V"
- board text added: "COM"
- board text added: "COMPRESSOR (L1-L2-L3), SSR OUTPUT (U-V-W)"
- board text added: "L"
- board text added: "MAINS (N-L1-L2-L3), SSR INPUT (R-S-T)"
- board text added: "R"
- board text added: "S"
- board text added: "SSR"
- board text added: "SSR 230V"
- board text added: "T"
- board text added: "U"
- board text added: "V"
- board text added: "W"
- board text removed: "COMPRESSOR"
- board text removed: "MAINS"
- board text removed: "WARNING HIGH VOLTAGE"

Commit message: WIP
Parts:
- C5: value 10M -> 10u
Changed lines of the file:
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@@
       (effects (font (size 1 1) (thickness 0.15)))
     )
-    (fp_text value 10M (at 0 1.75 270) (layer F.Fab)
+    (fp_text value 10u (at 0 1.75 270) (layer F.Fab)
       (effects (font (size 1 1) (thickness 0.15)))
     )

Commit message: WIP
Parts:
- added D5: SK22, Diodes_SMD:D_SMB, F.Cu at (172.5, 250.1)
Connections:
- R16 pad 2: +5V -> Net-(D5-Pad1)
- R17 pad 2: +5V -> Net-(D5-Pad1)
- R18 pad 2: +5V -> Net-(D5-Pad1)
Routing:
- net Net-(D5-Pad1): track 0.00 -> 15.9 mm
- net +5V: track 271.0 -> 255.2 mm
Changed lines of the file:
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@@
 (kicad_pcb (version 4) (host pcbnew 4.0.7-e2-6376~58~ubuntu16.04.1)
   (general
-    (links 224)
-    (no_connects 0)
+    (links 225)
+    (no_connects 3)
     (area 84.924999 119.924999 260.075001 240.075001)
     (thickness 1.6)
@@
     (tracks 829)
     (zones 0)
-    (modules 81)
-    (nets 63)
+    (modules 82)
+    (nets 64)
   )
   (page A3)
@@
   (net 61 /COMP_RELAY_PWR)
   (net 62 /COMP_RAMP)
+  (net 63 "Net-(D5-Pad1)")
   (net_class Default "This is the default net class."
     (clearance 0.199)
@@
     (add_net "Net-(D4-Pad5)")
     (add_net "Net-(D4-Pad6)")
+    (add_net "Net-(D5-Pad1)")
     (add_net "Net-(J3-Pad2)")
     (add_net "Net-(J3-Pad4)")
@@
       (net 60 /BACKUP_C))
     (pad 2 smd rect (at 3.1 0 270) (size 1 3.2) (layers F.Cu F.Paste F.Mask)
-      (net 9 +5V))
+      (net 63 "Net-(D5-Pad1)"))
     (model ${KISYS3DMOD}/Resistors_SMD.3dshapes/R_2512.wrl
       (at (xyz 0 0 0))
@@
       (net 60 /BACKUP_C))
     (pad 2 smd rect (at 3.1 0 270) (size 1 3.2) (layers F.Cu F.Paste F.Mask)
-      (net 9 +5V))
+      (net 63 "Net-(D5-Pad1)"))
     (model ${KISYS3DMOD}/Resistors_SMD.3dshapes/R_2512.wrl
       (at (xyz 0 0 0))
@@
       (net 60 /BACKUP_C))
     (pad 2 smd rect (at 3.1 0 270) (size 1 3.2) (layers F.Cu F.Paste F.Mask)
-      (net 9 +5V))
+      (net 63 "Net-(D5-Pad1)"))
     (model ${KISYS3DMOD}/Resistors_SMD.3dshapes/R_2512.wrl
       (at (xyz 0 0 0))
@@
       (xy 0.633952 -5.96402) (xy 0.746535 -5.366828)) (layer F.SilkS) (width 0.01))
   )
+  (module Diodes_SMD:D_SMB (layer F.Cu)
+    (at 172.5 250.075001)
+    (descr "Diode SMB (DO-214AA)")
+    (tags "Diode SMB (DO-214AA)")
+    (attr smd)
+    (fp_text reference D5 (at 0 -3) (layer F.SilkS)
+      (effects (font (size 1 1) (thickness 0.15)))
+    )
+    (fp_text value SK22 (at 0 3.1) (layer F.Fab)
+      (effects (font (size 1 1) (thickness 0.15)))
+    )
+    (fp_text user %R (at 0 -3) (layer F.Fab)
+      (effects (font (size 1 1) (thickness 0.15)))
+    )
+    (fp_line (start -3.55 -2.15) (end -3.55 2.15) (layer F.SilkS) (width 0.12))
+    (fp_line (start 2.3 2) (end -2.3 2) (layer F.Fab) (width 0.1))
+    (fp_line (start -2.3 2) (end -2.3 -2) (layer F.Fab) (width 0.1))
+    (fp_line (start 2.3 -2) (end 2.3 2) (layer F.Fab) (width 0.1))
+    (fp_line (start 2.3 -2) (end -2.3 -2) (layer F.Fab) (width 0.1))
+    (fp_line (start -3.65 -2.25) (end 3.65 -2.25) (layer F.CrtYd) (width 0.05))
+    (fp_line (start 3.65 -2.25) (end 3.65 2.25) (layer F.CrtYd) (width 0.05))
+    (fp_line (start 3.65 2.25) (end -3.65 2.25) (layer F.CrtYd) (width 0.05))
+    (fp_line (start -3.65 2.25) (end -3.65 -2.25) (layer F.CrtYd) (width 0.05))
+    (fp_line (start -0.64944 0.00102) (end -1.55114 0.00102) (layer F.Fab) (width 0.1))
+    (fp_line (start 0.50118 0.00102) (end 1.4994 0.00102) (layer F.Fab) (width 0.1))
+    (fp_line (start -0.64944 -0.79908) (end -0.64944 0.80112) (layer F.Fab) (width 0.1))
+    (fp_line (start 0.50118 0.75032) (end 0.50118 -0.79908) (layer F.Fab) (width 0.1))
+    (fp_line (start -0.64944 0.00102) (end 0.50118 0.75032) (layer F.Fab) (width 0.1))
+    (fp_line (start -0.64944 0.00102) (end 0.50118 -0.79908) (layer F.Fab) (width 0.1))
+    (fp_line (start -3.55 2.15) (end 2.15 2.15) (layer F.SilkS) (width 0.12))
+    (fp_line (start -3.55 -2.15) (end 2.15 -2.15) (layer F.SilkS) (width 0.12))
+    (pad 1 smd rect (at -2.15 0) (size 2.5 2.3) (layers F.Cu F.Paste F.Mask)
+      (net 63 "Net-(D5-Pad1)"))
+    (pad 2 smd rect (at 2.15 0) (size 2.5 2.3) (layers F.Cu F.Paste F.Mask)
+      (net 9 +5V))
+    (model ${KISYS3DMOD}/Diodes_SMD.3dshapes/D_SMB.wrl
+      (at (xyz 0 0 0))
+      (scale (xyz 1 1 1))
+      (rotate (xyz 0 0 0))
+    )
+  )
   (gr_text N (at 200 121.75 180) (layer F.SilkS)
     (effects (font (size 1.5 1.5) (thickness 0.3)))
@@
   (segment (start 174.515434 171.484566) (end 174.515434 183.803966) (width 0.6) (layer B.Cu) (net 9))
   (via (at 174.515434 184.440362) (size 0.9) (drill 0.6) (layers F.Cu B.Cu) (net 9))
-  (segment (start 179 167) (end 179 170.2) (width 0.6) (layer F.Cu) (net 9))
   (via (at 179 167) (size 0.9) (drill 0.6) (layers F.Cu B.Cu) (net 9))
   (segment (start 228 187) (end 203 187) (width 0.6) (layer B.Cu) (net 9))
@@
   (segment (start 187.300002 169) (end 185.000002 171.3) (width 0.6) (layer F.Cu) (net 9))
   (segment (start 185.000002 171.3) (end 181.2 171.3) (width 0.6) (layer F.Cu) (net 9))
-  (segment (start 181.2 171.3) (end 180.1 170.2) (width 0.6) (layer F.Cu) (net 9))
-  (segment (start 180.1 170.2) (end 179 170.2) (width 0.6) (layer F.Cu) (net 9))
-  (segment (start 174 170.2) (end 179 170.2) (width 0.6) (layer F.Cu) (net 9))
-  (segment (start 169 170.2) (end 174 170.2) (width 0.6) (layer F.Cu) (net 9))
   (segment (start 196.5 222.38) (end 196.5 224.885) (width 0.6) (layer F.Cu) (net 9))
   (segment (start 196.5 224.885) (end 196.5 230) (width 0.6) (layer F.Cu) (net 9))
@@
   (segment (start 236 126) (end 234.92 127.08) (width 0.4) (layer F.Cu) (net 62))
   (segment (start 234.92 130.38) (end 234.92 138) (width 0.4) (layer F.Cu) (net 62))
+  (segment (start 179 167) (end 179 170.2) (width 0.6) (layer F.Cu) (net 63))
+  (segment (start 181.2 171.3) (end 180.1 170.2) (width 0.6) (layer F.Cu) (net 63))
+  (segment (start 180.1 170.2) (end 179 170.2) (width 0.6) (layer F.Cu) (net 63))
+  (segment (start 174 170.2) (end 179 170.2) (width 0.6) (layer F.Cu) (net 63))
+  (segment (start 169 170.2) (end 174 170.2) (width 0.6) (layer F.Cu) (net 63))
   (zone (net 2) (net_name GND) (layer B.Cu) (hatch edge 0.508)
     (connect_pads (clearance 0.508))

Commit message: WIP
Parts:
- C2, C3: value 10u -> 1m; footprint Capacitors_SMD:C_0805 -> Capacitors_SMD:CP_Elec_8x10
- moved D5 81.4 mm to (187.2, 170.0)
- moved U1 3.91 mm to (187.2, 186.0)
- moved U2 3.89 mm to (175.0, 186.0)
- moved D1 3.70 mm to (190.0, 163.2)
- moved D2 3.70 mm to (184.0, 163.2)
- turned C2 to 180 degrees
- turned C3 to 180 degrees
Connections:
- C2 pad 1: GND -> /3V3_BACKUP
- C2 pad 2: /3V3_BACKUP -> GND
- C3 pad 1: GND -> +3V3
- C3 pad 2: +3V3 -> GND
Routing:
- net GND: track 106.8 -> 128.1 mm, vias 33 -> 31
- net /3V3_BACKUP: track 142.8 -> 130.5 mm
- net +5V: track 255.2 -> 245.9 mm, vias 7 -> 6
- net /COMP_RELAY: track 28.8 -> 23.1 mm, vias 2 -> 0
- net /COMP_RELAY_PWR: track 152.4 -> 157.2 mm
- net /BACKUP_C: track 66.1 -> 64.0 mm
- net Net-(D5-Pad1): track 15.9 -> 17.2 mm
- net +3V3: track 168.1 -> 167.4 mm
- net /5V_BACKUP: track 135.2 -> 135.4 mm, vias 6 -> 4
Other:
- board text added: "GWHP v1.2"
- board text removed: "GWHP v1.1"

Commit message: WIP
Parts:
- removed U4: Omega2, device.farm:Omega2+
- added J24: GS3, Connectors:GS3, F.Cu at (213.0, 166.0)
- added M1: NanoPi-Duo, device.farm:NanoPi-Duo, F.Cu at (235.5, 156.4)
- moved D1 8.15 mm to (196.2, 168.5), turned to 180 degrees
- moved C13 5.02 mm to (199.5, 153.5)
- moved D3 5.02 mm to (205.2, 168.5)
- moved D2 2.92 mm to (186.8, 162.5), turned to 180 degrees
- moved D5 1.58 mm to (186.7, 168.5)
Routing:
- net /RX0: track 6.93 -> 46.4 mm, vias 0 -> 2
- net /TX0: track 7.15 -> 43.5 mm, vias 0 -> 2
- net /ALERT: track 93.7 -> 115.6 mm
- net +5V: track 245.9 -> 263.4 mm, vias 6 -> 7
- net +3V3: track 167.4 -> 152.6 mm, vias 5 -> 2
- net /SCL: track 128.5 -> 140.0 mm, vias 2 -> 3
- net Net-(J24-Pad2): track 0.00 -> 8.67 mm
- net /COMP_RELAY_PWR: track 157.2 -> 149.5 mm, vias 1 -> 2
- net GND: track 128.1 -> 121.7 mm, vias 31 -> 29
- net /5V_BACKUP: track 135.4 -> 141.5 mm, vias 4 -> 2
- net /SDA: track 132.0 -> 138.2 mm
- net /USB-DP: track 7.24 -> 12.1 mm
- net /USB-DM: track 7.02 -> 11.4 mm
- net /BACKUP_C: track 64.0 -> 67.6 mm, vias 0 -> 3
- net /COMP_5V: track 345.8 -> 343.8 mm
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Other:
- board text added: "BACKUP"
- board text added: "BN"
- board text added: "GN"
- board text added: "NANOOK v1.3"
- board text added: "NO BACKUP"
- board text added: "WE"
- board text added: "YW"
- board text removed: "A1"
- board text removed: "A2"
- board text removed: "B1"
- board text removed: "B2"
- board text removed: "DEVICE.FARM"
- board text removed: "GWHP v1.2"
