File: board/nanook-mb.kicad_pcb (KiCad board)
At the start: 2 copper layers, 175 x 120 mm, 83 parts, among them J1 Power Switch, J10 Service, J11 Mains L3, J12 Mains N, J13 SSR 220, J14 SSR 0-5V, J15 Compressor L1, J16 Compressor L2, J17 Compressor L3, J18 SSR Output L1, J19 SSR Output L2, J2 Mains L1, J20 SSR Output L3, J21 SSR Input L1, J22 SSR Input L2, J23 SSR Input L3, J24 GS3, J3 AUX, J4 E2V, J5 LPS, J6 Pump Cold Side, J7 Pump Hot Side, J8 HPS, J9 Mains L2, K1 RELAY_2, K2 RELAY_2, K3 RELAY_2, M1 NanoPi-Duo, T1 BC817, U1 NCP1117-3.3_SOT223, U2 NCP1117-3.3_SOT223, U3 Mean Well PM-15-5, U5 STM32F030K6Tx, U6 DRV8833, U7 MCP4706A0T-E/CH, U8 G3MB-5V-SSR, U9 G3MB-5V-SSR, X1 SWD, X2 I2C Cold Side, X3 I2C Hot Side, X4 I2C Aux

Commit message: Kicad 5
Connections:
- M1 pad 1: (no net) -> Net-(M1-Pad1)
- M1 pad 10: (no net) -> Net-(M1-Pad10)
- M1 pad 11: (no net) -> Net-(M1-Pad11)
- M1 pad 12: (no net) -> Net-(M1-Pad12)
- M1 pad 14: (no net) -> Net-(M1-Pad14)
- M1 pad 2: (no net) -> Net-(M1-Pad2)
- M1 pad 23: (no net) -> Net-(M1-Pad23)
- M1 pad 24: (no net) -> Net-(M1-Pad24)
- M1 pad 25: (no net) -> Net-(M1-Pad25)
- M1 pad 26: (no net) -> Net-(M1-Pad26)
- M1 pad 27: (no net) -> Net-(M1-Pad27)
- M1 pad 28: (no net) -> Net-(M1-Pad28)
- M1 pad 29: (no net) -> Net-(M1-Pad29)
- M1 pad 3: (no net) -> Net-(M1-Pad3)
- M1 pad 30: (no net) -> Net-(M1-Pad30)
- M1 pad 31: (no net) -> Net-(M1-Pad31)
- M1 pad 32: (no net) -> Net-(M1-Pad32)
- M1 pad 4: (no net) -> Net-(M1-Pad4)
- M1 pad 5: (no net) -> Net-(M1-Pad5)
- M1 pad 6: (no net) -> Net-(M1-Pad6)
- M1 pad 9: (no net) -> Net-(M1-Pad9)
- U7 pad 6: (no net) -> Net-(U7-Pad6)

Commit message: WIP
Parts:
- C10, C11, C12, C4, C5, C6, C7, C8, C9: footprint Capacitors_SMD:C_0805 -> Capacitor_SMD:C_0805_2012Metric
- C2, C3: footprint Capacitors_SMD:CP_Elec_8x10 -> Capacitor_SMD:CP_Elec_8x10
- D1, D2, D3, D5: footprint Diodes_SMD:D_SMB -> Diode_SMD:D_SMB
- J10: footprint Pin_Headers:Pin_Header_Straight_1x06_Pitch2.54mm -> Connector_PinHeader_2.54mm:PinHeader_1x06_P2.54mm_Vertical
- J24: footprint Connectors:GS3 -> Jumper:SolderJumper-3_P1.3mm_Open_Pad1.0x1.5mm
- J3: footprint Pin_Headers:Pin_Header_Straight_2x05_Pitch2.54mm -> Connector_PinHeader_2.54mm:PinHeader_2x05_P2.54mm_Vertical
- R1, R10, R11, R12, R13, R14, R15, R2, R3, R4, R5, R6, R7, R8, R9: footprint Resistors_SMD:R_0805 -> Resistor_SMD:R_0805_2012Metric
- R16, R17, R18: footprint Resistors_SMD:R_2512 -> Resistor_SMD:R_2512_6332Metric
- T1: footprint TO_SOT_Packages_SMD:SOT-23 -> Package_TO_SOT_SMD:SOT-23
- U1, U2: footprint TO_SOT_Packages_SMD:SOT-223-3Lead_TabPin2 -> Package_TO_SOT_SMD:SOT-223-3_TabPin2
- U5: footprint Housings_QFP:LQFP-32_7x7mm_Pitch0.8mm -> Package_QFP:LQFP-32_7x7mm_P0.8mm
- U7: footprint TO_SOT_Packages_SMD:SOT-23-6 -> Package_TO_SOT_SMD:SOT-23-6
- turned J24 to 270 degrees
