File: board/nanook-mb.kicad_pcb (KiCad board)
At the start: 2 copper layers, 175 x 120 mm, 83 parts, among them J1 Power Switch, J10 Service, J11 Mains L3, J12 Mains N, J13 SSR 220, J14 SSR 0-5V, J15 Compressor L1, J16 Compressor L2, J17 Compressor L3, J18 SSR Output L1, J19 SSR Output L2, J2 Mains L1, J20 SSR Output L3, J21 SSR Input L1, J22 SSR Input L2, J23 SSR Input L3, J24 GS3, J3 AUX, J4 E2V, J5 LPS, J6 Pump Cold Side, J7 Pump Hot Side, J8 HPS, J9 Mains L2, K1 RELAY_2, K2 RELAY_2, K3 RELAY_2, M1 NanoPi-Duo, T1 BC817, U1 NCP1117-3.3_SOT223, U2 NCP1117-3.3_SOT223, U3 Mean Well PM-15-5, U5 STM32F030K6Tx, U6 DRV8833, U7 MCP4706A0T-E/CH, U8 G3MB-5V-SSR, U9 G3MB-5V-SSR, X1 SWD, X2 I2C Cold Side, X3 I2C Hot Side, X4 I2C Aux

Commit message: WIP
Parts:
- C1, C13: footprint device.farm:BCE005R5C205FS -> Drake:BCE005R5C205FS
- D4: footprint device.farm:LED_RGB_5050-6 -> Drake:LED_RGB_5050-6
- J1, J13, J14, J5, J6, J7, J8: footprint device.farm:DG142R-2-5.08 -> Drake:DG142R-2-5.08
- J11, J12, J15, J16, J17, J18, J19, J2, J20, J21, J22, J23, J9: footprint device.farm:Tab-6.3 -> Drake:Tab-6.3
- J4: footprint device.farm:DG142R-4-5.08 -> Drake:DG142R-4-5.08
- K1, K2, K3: footprint device.farm:RT314_Relay -> Drake:RT314_Relay
- M1: footprint device.farm:NanoPi-Duo -> Drake:NanoPi-Duo
- S1: footprint device.farm:SB2P -> Drake:SB2P
- U3: footprint device.farm:Mean-Well-PM-15-5 -> Drake:Mean-Well-PM-15-5
- U6: footprint device.farm:TSSOP-16_4.4x5mm_Pitch0.65mm-EP -> Drake:TSSOP-16_4.4x5mm_Pitch0.65mm-EP
- U8, U9: footprint device.farm:G3MB-SSR -> Drake:G3MB-SSR
- X1: footprint device.farm:SWD -> Drake:SWD
- X2, X3, X4: footprint device.farm:Micro-Match-FOB-6 -> Drake:Micro-Match-FOB-6
Changed lines of the file:
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@@
     )
   )
-  (module device.farm:RT314_Relay (layer F.Cu)
+  (module Drake:RT314_Relay (layer F.Cu)
     (at 185 147.38 180)
     (fp_text reference K3 (at -2 4.38 180) (layer F.SilkS)
@@
     )
   )
-  (module device.farm:RT314_Relay (layer F.Cu)
+  (module Drake:RT314_Relay (layer F.Cu)
     (at 115 147.38 180)
     (fp_text reference K1 (at -2 4.38 180) (layer F.SilkS)
@@
     )
   )
-  (module device.farm:RT314_Relay (layer F.Cu)
+  (module Drake:RT314_Relay (layer F.Cu)
     (at 150 147.38 180)
     (fp_text reference K2 (at -2 4.38 180) (layer F.SilkS)
@@
     )
   )
-  (module device.farm:BCE005R5C205FS (layer F.Cu)
+  (module Drake:BCE005R5C205FS (layer F.Cu)
     (at 199.5 153.5 180)
     (fp_text reference C13 (at 0 11.5 180) (layer F.SilkS)
@@
     )
   )
-  (module device.farm:BCE005R5C205FS (layer F.Cu)
+  (module Drake:BCE005R5C205FS (layer F.Cu)
     (at 216 132 180)
     (fp_text reference C1 (at 12 0 180) (layer F.SilkS)
@@
     )
   )
-  (module device.farm:DG142R-2-5.08 (layer F.Cu)
+  (module Drake:DG142R-2-5.08 (layer F.Cu)
     (at 187.54 139.778 180)
     (fp_text reference J1 (at 5.334 15.494 180) (layer F.SilkS) hide
@@
     )
   )
-  (module device.farm:DG142R-4-5.08 (layer F.Cu)
+  (module Drake:DG142R-4-5.08 (layer F.Cu)
     (at 224.22 220.602)
     (fp_text reference J4 (at 5.334 15.494) (layer F.SilkS) hide
@@
     )
   )
-  (module device.farm:DG142R-2-5.08 (layer F.Cu)
+  (module Drake:DG142R-2-5.08 (layer F.Cu)
     (at 193.96 220.602)
     (fp_text reference J5 (at 5.334 15.494) (layer F.SilkS) hide
@@
     )
   )
-  (module device.farm:DG142R-2-5.08 (layer F.Cu)
+  (module Drake:DG142R-2-5.08 (layer F.Cu)
     (at 163.96 220.602)
     (fp_text reference J6 (at 5.334 15.494) (layer F.SilkS) hide
@@
     )
   )
-  (module device.farm:DG142R-2-5.08 (layer F.Cu)
+  (module Drake:DG142R-2-5.08 (layer F.Cu)
     (at 178.96 220.602)
     (fp_text reference J7 (at 5.334 15.494) (layer F.SilkS) hide
@@
     )
   )
-  (module device.farm:DG142R-2-5.08 (layer F.Cu)
+  (module Drake:DG142R-2-5.08 (layer F.Cu)
     (at 208.96 220.602)
     (fp_text reference J8 (at 5.334 15.494) (layer F.SilkS) hide
@@
     )
   )
-  (module device.farm:SB2P (layer F.Cu)
+  (module Drake:SB2P (layer F.Cu)
     (at 220 176.984 90)
     (fp_text reference S1 (at -0.016 3 180) (layer F.SilkS)
@@
       (net 39 "Net-(S1-Pad1)"))
   )
-  (module device.farm:Mean-Well-PM-15-5 (layer F.Cu)
+  (module Drake:Mean-Well-PM-15-5 (layer F.Cu)
     (at 125 190 270)
     (fp_text reference U3 (at -7 39 270) (layer F.SilkS)
@@
     )
   )
-  (module device.farm:G3MB-SSR (layer F.Cu)
+  (module Drake:G3MB-SSR (layer F.Cu)
     (at 171.58 203.84 270)
     (fp_text reference U8 (at -11.84 -5.42) (layer F.SilkS)
@@
     )
   )
-  (module device.farm:G3MB-SSR (layer F.Cu)
+  (module Drake:G3MB-SSR (layer F.Cu)
     (at 186.58 203.84 270)
     (fp_text reference U9 (at -11.84 -5.42) (layer F.SilkS)
@@
     )
   )
-  (module device.farm:SWD (layer F.Cu)
+  (module Drake:SWD (layer F.Cu)
     (at 231.14 175.26 180)
     (fp_text reference X1 (at 0 2.54 180) (layer F.SilkS) hide
@@
       (net 48 /SWDIO))
   )
-  (module device.farm:Micro-Match-FOB-6 (layer F.Cu)
+  (module Drake:Micro-Match-FOB-6 (layer F.Cu)
     (at 252 211)
     (fp_text reference X2 (at -6 0) (layer F.SilkS) hide
@@
     )
   )
-  (module device.farm:Micro-Match-FOB-6 (layer F.Cu)
+  (module Drake:Micro-Match-FOB-6 (layer F.Cu)
     (at 252 199)
     (fp_text reference X3 (at -6 0) (layer F.SilkS) hide
@@
     )
   )
-  (module device.farm:Micro-Match-FOB-6 (layer F.Cu)
+  (module Drake:Micro-Match-FOB-6 (layer F.Cu)
     (at 252 187)
     (fp_text reference X4 (at -6 0) (layer F.SilkS) hide
@@
     )
   )
-  (module device.farm:LED_RGB_5050-6 (layer F.Cu)
+  (module Drake:LED_RGB_5050-6 (layer F.Cu)
     (at 239.6 193 180)
     (descr http://cdn.sparkfun.com/datasheets/Components/LED/5060BRG4.pdf)
@@
     )
   )
-  (module device.farm:TSSOP-16_4.4x5mm_Pitch0.65mm-EP (layer F.Cu)
+  (module Drake:TSSOP-16_4.4x5mm_Pitch0.65mm-EP (layer F.Cu)
     (at 232.6 207.6)
     (descr "16-Lead Plastic Thin Shrink Small Outline (ST)-4.4 mm Body [TSSOP] (see Microchip Packaging Specification 00000049BS.pdf)")
@@
     )
   )
-  (module device.farm:DG142R-2-5.08 (layer F.Cu)
+  (module Drake:DG142R-2-5.08 (layer F.Cu)
     (at 202.54 139.778 180)
     (fp_text reference J13 (at 5.334 15.494 180) (layer F.SilkS) hide
@@
     )
   )
-  (module device.farm:DG142R-2-5.08 (layer F.Cu)
+  (module Drake:DG142R-2-5.08 (layer F.Cu)
     (at 242.54 139.778 180)
     (fp_text reference J14 (at -3.46 15.778 180) (layer F.SilkS) hide
@@
     )
   )
-  (module device.farm:Tab-6.3 (layer F.Cu)
+  (module Drake:Tab-6.3 (layer F.Cu)
     (at 115 227.46 90)
     (fp_text reference J15 (at 0 3.5 90) (layer F.SilkS) hide
@@
     )
   )
-  (module device.farm:Tab-6.3 (layer F.Cu)
+  (module Drake:Tab-6.3 (layer F.Cu)
     (at 135 227.46 90)
     (fp_text reference J16 (at 0 3.5 90) (layer F.SilkS) hide
@@
     )
   )
-  (module device.farm:Tab-6.3 (layer F.Cu)
+  (module Drake:Tab-6.3 (layer F.Cu)
     (at 155 227.46 90)
     (fp_text reference J17 (at 0 3.5 90) (layer F.SilkS) hide
@@
     )
   )
-  (module device.farm:Tab-6.3 (layer F.Cu)
+  (module Drake:Tab-6.3 (layer F.Cu)
     (at 105 227.46 90)
     (fp_text reference J18 (at 0 3.5 90) (layer F.SilkS) hide
@@
     )
   )
-  (module device.farm:Tab-6.3 (layer F.Cu)
+  (module Drake:Tab-6.3 (layer F.Cu)
     (at 125 227.46 90)
     (fp_text reference J19 (at 0 3.5 90) (layer F.SilkS) hide
@@
     )
   )
-  (module device.farm:Tab-6.3 (layer F.Cu)
+  (module Drake:Tab-6.3 (layer F.Cu)
     (at 145 227.46 90)
     (fp_text reference J20 (at 0 3.5 90) (layer F.SilkS) hide
@@
     )
   )
-  (module device.farm:Tab-6.3 (layer F.Cu)
+  (module Drake:Tab-6.3 (layer F.Cu)
     (at 105 132.46 90)
     (fp_text reference J21 (at 0 3.5 90) (layer F.SilkS) hide
@@
     )
   )
-  (module device.farm:Tab-6.3 (layer F.Cu)
+  (module Drake:Tab-6.3 (layer F.Cu)
     (at 125 132.46 90)
     (fp_text reference J22 (at 0 3.5 90) (layer F.SilkS) hide
@@
     )
   )
-  (module device.farm:Tab-6.3 (layer F.Cu)
+  (module Drake:Tab-6.3 (layer F.Cu)
     (at 145 132.46 90)
     (fp_text reference J23 (at 0 3.5 90) (layer F.SilkS) hide
@@
     )
   )
-  (module device.farm:Tab-6.3 (layer F.Cu)
+  (module Drake:Tab-6.3 (layer F.Cu)
     (at 115 132.46 90)
     (fp_text reference J2 (at 0 3.5 90) (layer F.SilkS) hide
@@
     )
   )
-  (module device.farm:Tab-6.3 (layer F.Cu)
+  (module Drake:Tab-6.3 (layer F.Cu)
     (at 135 132.46 90)
     (fp_text reference J9 (at 0 3.5 90) (layer F.SilkS) hide
@@
     )
   )
-  (module device.farm:Tab-6.3 (layer F.Cu)
+  (module Drake:Tab-6.3 (layer F.Cu)
     (at 155 132.46 90)
     (fp_text reference J11 (at 0 3.5 90) (layer F.SilkS) hide
@@
     )
   )
-  (module device.farm:Tab-6.3 (layer F.Cu)
+  (module Drake:Tab-6.3 (layer F.Cu)
     (at 169 133.46 270)
     (fp_text reference J12 (at 0 3.5 270) (layer F.SilkS) hide
@@
     )
   )
-  (module device.farm:NanoPi-Duo (layer F.Cu)
+  (module Drake:NanoPi-Duo (layer F.Cu)
     (at 235.54 156.430248)
     (fp_text reference M1 (at 0 0) (layer F.SilkS)

Commit message: WIP
Other:
- net class Default removed
- net class HC removed
- net class LC removed
- net class PWR removed
- board text added: "DC25"
